Commit message: remap mode of velocity and pecent output

File: description/ros2_control/diffbot.ros2_control.xacro (robot description, xacro)
@@ -6,6 +6,7 @@
         <!-- <plugin>diffdrive_arduino/DiffDriveArduinoHardware</plugin> -->
         <plugin>ros_phoenix/PhoenixBridge</plugin>
-        <param name="left_wheel_name">left_wheel_joint</param>
-        <param name="right_wheel_name">right_wheel_joint</param>
+        <!-- <plugin>ros_phoenix/PhoenixSystem</plugin> -->
+        <!-- <param name="left_wheel_name">left_wheel_joint</param>
+        <param name="right_wheel_name">right_wheel_joint</param> -->
         <!-- <param name="loop_rate">30</param> -->
         <!-- <param name="device">/dev/serial/by-path/platform-fd500000.pcie-pci-0000:01:00.0-usb-0:1.3:1.0-port0</param> -->
@@ -23,5 +24,5 @@
         <state_interface name="velocity"/>
       </joint>
-      <joint name="${prefix}right_wheel_joint">
+    <joint name="${prefix}right_wheel_joint">
         <command_interface name="velocity"/>
         <state_interface name="position"/>

File: description/urdf/diffbot.urdf.xacro (robot description, xacro)
@@ -1,16 +0,0 @@
-<?xml version="1.0"?>
-<!-- Basic differential drive mobile base -->
-<robot xmlns:xacro="http://www.ros.org/wiki/xacro" name="diffdrive_robot">
-  <xacro:arg name="prefix" default="" />
-  <!-- <xacro:include filename="$(find diffdrive_arduino)/urdf/diffbot_description.urdf.xacro" /> -->
-  <xacro:include filename="$(find ros_phoenix)/urdf/diffbot_description.urdf.xacro" />
-  <!-- Import Rviz colors -->
-  <!-- <xacro:include filename="$(find diffdrive_arduino)/urdf/diffbot.materials.xacro" /> -->
-  <xacro:include filename="$(find ros_phoenix)/urdf/diffbot.materials.xacro" />
-  <!-- Import diffbot ros2_control description -->
-  <!-- <xacro:include filename="$(find diffdrive_arduino)/ros2_control/diffbot.ros2_control.xacro" /> -->
-  <xacro:include filename="$(find ros_phoenix)/ros2_control/phoenix_bridge_example.ros2_control.xacro" />
-  <xacro:diffbot prefix="$(arg prefix)" />
-  <xacro:diffbot_ros2_control
-    name="DiffBot" prefix="$(arg prefix)" />
-</robot>

Commit message: update 03/09/2024

File: description/ros2_control/diffbot.ros2_control.xacro (robot description, xacro)
@@ -2,32 +2,75 @@
 <robot xmlns:xacro="http://www.ros.org/wiki/xacro">
   <xacro:macro name="diffbot_ros2_control" params="name prefix">
-    <ros2_control name="${name}" type="system">
-      <hardware>
-        <!-- <plugin>diffdrive_arduino/DiffDriveArduinoHardware</plugin> -->
-        <plugin>ros_phoenix/PhoenixBridge</plugin>
-        <!-- <plugin>ros_phoenix/PhoenixSystem</plugin> -->
-        <!-- <param name="left_wheel_name">left_wheel_joint</param>
-        <param name="right_wheel_name">right_wheel_joint</param> -->
-        <!-- <param name="loop_rate">30</param> -->
-        <!-- <param name="device">/dev/serial/by-path/platform-fd500000.pcie-pci-0000:01:00.0-usb-0:1.3:1.0-port0</param> -->
-        <!-- <param name="baud_rate">57600</param> -->
-        <!-- <param name="timeout_ms">1000</param> -->
-        <!-- <param name="enc_counts_per_rev">3436</param> -->
-        <!-- <param name="pid_p">20</param> -->
-        <!-- <param name="pid_d">12</param> -->
-        <!-- <param name="pid_i">0</param> -->
-        <!-- <param name="pid_o">50</param> -->
-      </hardware>
-      <joint name="${prefix}left_wheel_joint">
-        <command_interface name="velocity"/>
-        <state_interface name="position"/>
-        <state_interface name="velocity"/>
-      </joint>
-    <joint name="${prefix}right_wheel_joint">
-        <command_interface name="velocity"/>
-        <state_interface name="position"/>
-        <state_interface name="velocity"/>
-      </joint>
-    </ros2_control>
+    <xacro:unless value="$(arg sim_mode)">
+      <ros2_control name="${name}" type="system">
+        <hardware>
+          <!-- <plugin>diffdrive_arduino/DiffDriveArduinoHardware</plugin> -->
+          <plugin>ros_phoenix/PhoenixBridge</plugin>
+          <!-- <plugin>ros_phoenix/PhoenixSystem</plugin> -->
+          <!-- <param name="left_wheel_name">left_wheel_joint</param>
+          <param name="right_wheel_name">right_wheel_joint</param> -->
+          <!-- <param name="loop_rate">30</param> -->
+          <!-- <param name="device">/dev/serial/by-path/platform-fd500000.pcie-pci-0000:01:00.0-usb-0:1.3:1.0-port0</param> -->
+          <!-- <param name="baud_rate">57600</param> -->
+          <!-- <param name="timeout_ms">1000</param> -->
+          <!-- <param name="enc_counts_per_rev">3436</param> -->
+          <!-- <param name="pid_p">20</param> -->
+          <!-- <param name="pid_d">12</param> -->
+          <!-- <param name="pid_i">0</param> -->
+          <!-- <param name="pid_o">50</param> -->
+        </hardware>
+        <joint name="${prefix}left_wheel_joint">
+          <command_interface name="velocity"/>
+          <state_interface name="position"/>
+          <state_interface name="velocity"/>
+        </joint>
+        <joint name="${prefix}right_wheel_joint">
+          <command_interface name="velocity"/>
+          <state_interface name="position"/>
+          <state_interface name="velocity"/>
+        </joint>
+      </ros2_control>
+    </xacro:unless>
+    <xacro:if value= "$(arg sim_mode)">
+      <ros2_control name="GazeboSystem" type="system">
+        <hardware>
+            <plugin>gazebo_ros2_control/GazeboSystem</plugin>
+        </hardware>
+        <joint name="${prefix}left_wheel_joint">
+          <command_interface name="velocity"/>
+          <state_interface name="position"/>
+          <state_interface name="velocity"/>
+        </joint>
+        <joint name="${prefix}right_wheel_joint">
+          <command_interface name="velocity"/>
+          <state_interface name="position"/>
+          <state_interface name="velocity"/>
+        </joint>
+      </ros2_control>
+      <gazebo reference="imu_link">
+        <gravity>true</gravity>
+        <sensor name="imu_sensor" type="imu">
+          <always_on>true</always_on>
+          <update_rate>100</update_rate>
+          <visualize>true</visualize>
+          <plugin filename="libgazebo_ros_imu_sensor.so" name="imu_plugin">
+            <ros>
+                <remapping>~/out:=imu/data_raw</remapping>
+            </ros>
+            <topicName>imu</topicName>
+            <bodyName>imu_link</bodyName>
+            <update_rate>100</update_rate>
+            <frameName>imu_link</frameName>
+            <initialOrientationAsReference>false</initialOrientationAsReference>
+          </plugin>
+        </sensor>
+      </gazebo>
+    </xacro:if>
+    <gazebo>
+        <plugin name="gazebo_ros2_control" filename="libgazebo_ros2_control.so">
+            <parameters>$(find ros_phoenix)/config/diffbot_controllers.yaml</parameters>
+            <parameters>$(find ros_phoenix)/config/gaz_ros2_ctl_use_sim.yaml</parameters>
+        </plugin>
+    </gazebo>
   </xacro:macro>
 </robot>

File: description/urdf/diffbot.urdf.xacro (robot description, xacro)
@@ -0,0 +1,18 @@
+<?xml version="1.0"?>
+<!-- Basic differential drive mobile base -->
+<robot xmlns:xacro="http://www.ros.org/wiki/xacro" name="diffdrive_robot">
+  <xacro:arg name="prefix" default="" />
+  <xacro:arg name="sim_mode" default="false"/>
+  <!-- <xacro:include filename="$(find diffdrive_arduino)/urdf/diffbot_description.urdf.xacro" /> -->
+  <xacro:include filename="$(find ros_phoenix)/urdf/diffbot_description.urdf.xacro" />
+  <!-- <xacro:include filename="$(find ros_phoenix)/urdf/robot_core.urdf.xacro" /> -->
+  <!-- Import Rviz colors -->
+  <!-- <xacro:include filename="$(find diffdrive_arduino)/urdf/diffbot.materials.xacro" /> -->
+  <xacro:include filename="$(find ros_phoenix)/urdf/diffbot.materials.xacro" />
+  <!-- Import diffbot ros2_control description -->
+  <!-- <xacro:include filename="$(find diffdrive_arduino)/ros2_control/diffbot.ros2_control.xacro" /> -->
+  <xacro:include filename="$(find ros_phoenix)/ros2_control/diffbot.ros2_control.xacro" />
+  <xacro:diffbot prefix="$(arg prefix)" />
+  <xacro:diffbot_ros2_control
+    name="DiffBot" prefix="$(arg prefix)"/>
+</robot>

File: description/urdf/robot_core.urdf.xacro (robot description, xacro)
@@ -1,9 +1,10 @@
 <?xml version="1.0"?>
 <robot xmlns:xacro="http://www.ros.org/wiki/xacro" >
-    <!-- the copy of robot_core_1 urdf -->
     <xacro:macro name="diffbot" params="prefix">
     <xacro:include filename="inertial_macros.xacro"/>
     <xacro:include filename="lidar.xacro" />
     <xacro:include filename="depth_camera.xacro"/>
+    <!-- inlucde bracket -->
+    <!-- <xacro:include filename="$(find ros_phoenix)/urdf/brackets.xacro" /> -->
     <xacro:property name="chassis_length" value="1.35" />
     <xacro:property name="chassis_width" value="0.5" />
@@ -22,9 +23,15 @@
     <link name="base_link">
     </link>
+    <joint name="imu_joint" type="fixed">
+        <parent link="base_footprint" />
+        <child link="imu_link" />
+        <origin xyz="0 0.05 ${wheel_offset_x+0.042}" rpy="0 0 0" />
+    </joint>
+    <link name="imu_link" />
     <!-- BASE_FOOTPRINT LINK -->
     <joint name="base_footprint_joint" type="fixed">
     	<parent link="base_link"/>
     	<child link="base_footprint"/>
-    	<origin xyz="0 0 0" rpy="0 0 0"/>
+    	<origin xyz="0 0 0" rpy="${pi} ${pi} 0"/>
     </joint>
     <link name="base_footprint">
@@ -32,5 +39,5 @@
     <!-- CHASSIS LINK -->
     <joint name="chassis_joint" type="fixed">
-        <parent link="base_link"/>
+        <parent link="base_footprint"/>
         <child link="chassis"/>
         <origin xyz="${-wheel_offset_x} 0 ${-wheel_offset_z}"/>
@@ -59,7 +66,7 @@
     <!-- BACK LEFT WHEEL LINK -->
     <joint name="left_wheel_joint" type="continuous">
-        <parent link="base_link"/>
+        <parent link="base_footprint"/>
         <child link="left_wheel"/>
-        <origin xyz="${caster_wheel_offset_x-0.1}  ${wheel_offset_y} 0" rpy="-${pi/2} 0 0" />
+        <origin xyz="0  ${wheel_offset_y} 0" rpy="-${pi/2} 0 ${pi}" />
         <axis xyz="0 0 1"/>
     </joint>
@@ -85,7 +92,7 @@
     <!-- BACK RIGHT WHEEL LINK -->
     <joint name="right_wheel_joint" type="continuous">
-        <parent link="base_link"/>
+        <parent link="base_footprint"/>
         <child link="right_wheel"/>
-        <origin xyz="${caster_wheel_offset_x-0.1} ${-wheel_offset_y} 0" rpy="${pi/2} 0 0" />
+        <origin xyz="0 ${-wheel_offset_y} 0" rpy="${pi/2} 0 ${-pi}" />
         <axis xyz="0 0 -1"/>
     </joint>
@@ -113,5 +120,5 @@
         <parent link="chassis"/>
         <child link="front_left_wheel"/>
-        <origin xyz="0.1 ${wheel_offset_y} ${wheel_offset_z}" rpy="-${pi/2} 0 0" />
+        <origin xyz="${caster_wheel_offset_x} ${wheel_offset_y} ${wheel_offset_z}" rpy="-${pi/2} 0 0" />
         <axis xyz="0 0 1"/>
     </joint>
@@ -141,5 +148,5 @@
         <parent link="chassis"/>
         <child link="front_right_wheel"/>
-        <origin xyz="0.1 ${-wheel_offset_y} ${wheel_offset_z}" rpy="${pi/2} 0 0" />
+        <origin xyz="${caster_wheel_offset_x} ${-wheel_offset_y} ${wheel_offset_z}" rpy="${pi/2} 0 0" />
         <axis xyz="0 0 -1"/>
     </joint>
@@ -165,9 +172,37 @@
         <mu2 value="0.001"/>
     </gazebo>
+    <!-- TOWER -->
+    <!-- Needs to be 0.510m tall -->
+    <joint name="tower" type="fixed">
+        <parent link="base_footprint"/>
+        <child link="tower"/>
+        <origin xyz="0.4615 0 0"/>
+    </joint>
+    <link name="tower">
+        <visual>
+            <origin xyz="0 0 0.025"/>
+            <geometry>
+                <box size="0.05 0.5 0.05"/>
+            </geometry>
+            <material name="orange"/>
+        </visual>
+        <collision>
+            <origin xyz="0 0 0.025"/>
+            <geometry>
+                <box size="0.05 0.5 0.05"/>
+            </geometry>
+        </collision>
+        <xacro:inertial_box mass="0.5" x="0.05" y="0.5" z="0.05">
+            <origin xyz="0 0 0.025" rpy="0 0 0"/>
+        </xacro:inertial_box>
+    </link>
+    <gazebo reference="tower">
+        <material>Gazebo/White</material>
+    </gazebo>
     <!-- MOTOR AND GEARBOX LINK -->
     <joint name="motor_joint" type="fixed">
-        <parent link="base_link"/>
+        <parent link="base_footprint"/>
         <child link="motor"/>
-        <origin xyz="${caster_wheel_offset_x-0.1} 0 0"/>
+        <origin xyz="0 0 0"/>
     </joint>
     <link name="motor">
@@ -192,36 +227,8 @@
         <material>Gazebo/Orange</material>
     </gazebo>
-    <!-- TOWER -->
-    <!-- Needs to be 0.510m tall -->
-    <joint name="tower" type="fixed">
-        <parent link="base_link"/>
-        <child link="tower"/>
-        <origin xyz="0.4615 0 0"/>
-    </joint>
-    <link name="tower">
-        <visual>
-            <origin xyz="0 0 0.025"/>
-            <geometry>
-                <box size="0.05 0.5 0.05"/>
-            </geometry>
-            <material name="orange"/>
-        </visual>
-        <collision>
-            <origin xyz="0 0 0.025"/>
-            <geometry>
-                <box size="0.05 0.5 0.05"/>
-            </geometry>
-        </collision>
-        <xacro:inertial_box mass="0.5" x="0.05" y="0.5" z="0.05">
-            <origin xyz="0 0 0.025" rpy="0 0 0"/>
-        </xacro:inertial_box>
-    </link>
-    <gazebo reference="tower">
-        <material>Gazebo/White</material>
-    </gazebo>
-    <!-- TOWER HEIGHT LEFT -->
+        <!-- TOWER HEIGHT LEFT -->
     <!-- Needs to be 0.510m tall -->
     <joint name="tower_up_left" type="fixed">
-        <parent link="base_link"/>
+        <parent link="base_footprint"/>
         <child link="tower_up_left"/>
         <origin xyz="0.4615 0 0"/>
@@ -248,5 +255,5 @@
     <!-- Needs to be 0.510m tall -->
     <joint name="tower_up_right" type="fixed">
-        <parent link="base_link"/>
+        <parent link="base_footprint"/>
         <child link="tower_up_right"/>
         <origin xyz="0.4615 0 0"/>
@@ -273,5 +280,5 @@
     <!-- Needs to be 0.510m tall -->
     <joint name="tower_top" type="fixed">
-        <parent link="base_link"/>
+        <parent link="base_footprint"/>
         <child link="tower_top"/>
         <origin xyz="0.4615 0 0"/>
@@ -295,4 +302,78 @@
         </xacro:inertial_box>
     </link>
+    <!-- TOWER HEIGHT LEFT MOTOR -->
+    <joint name="tower_motor_left" type="fixed">
+        <parent link="base_footprint"/>
+        <child link="tower_motor_left"/>
+        <origin xyz="0 0 0"/>
+    </joint>
+    <link name="tower_motor_left">
+        <visual>
+            <origin xyz="0 -0.24 ${wheel_offset_x/2}"/>
+            <geometry>
+                <box size="0.05 0.02 ${wheel_offset_x}"/>
+            </geometry>
+            <material name="orange"/>
+        </visual>
+        <collision>
+            <origin xyz="0 -0.24 ${wheel_offset_x/2}"/>
+            <geometry>
+                <box size="0.05 0.02 ${wheel_offset_x}"/>
+            </geometry>
+        </collision>
+        <xacro:inertial_box mass="0.5" x="0.05" y="0.02" z="${wheel_offset_x}">
+            <origin xyz="0 -0.24 ${wheel_offset_x/2}" rpy="0 0 0"/>
+        </xacro:inertial_box>
+    </link>
+    <!-- TOWER HEIGHT RIGHT-->
+    <!-- Needs to be 0.510m tall -->
+    <joint name="tower_motor_right" type="fixed">
+        <parent link="base_footprint"/>
+        <child link="tower_motor_right"/>
+        <origin xyz="0 0 0"/>
+    </joint>
+    <link name="tower_motor_right">
+        <visual>
+            <origin xyz="0 0.24 ${wheel_offset_x/2}"/>
+            <geometry>
+                <box size="0.05 0.02 ${wheel_offset_x}"/>
+            </geometry>
+            <material name="orange"/>
+        </visual>
+        <collision>
+            <origin xyz="0 0.24 ${wheel_offset_x/2}"/>
+            <geometry>
+                <box size="0.05 0.02 ${wheel_offset_x}"/>
+            </geometry>
+        </collision>
+        <xacro:inertial_box mass="0.5" x="0.05" y="0.02" z="${wheel_offset_x}">
+            <origin xyz="0 0.24 ${wheel_offset_x/2}" rpy="0 0 0"/>
+        </xacro:inertial_box>
+    </link>
+    <!-- TOWER motor TOP -->
+    <!-- Needs to be 0.510m tall -->
+    <joint name="tower_motor_top" type="fixed">
+        <parent link="base_footprint"/>
+        <child link="tower_motor_top"/>
+        <origin xyz="0 0 0"/>
+    </joint>
+    <link name="tower_motor_top">
+        <visual>
+            <origin xyz="0 0 ${wheel_offset_x}"/>
+            <geometry>
+                <box size="0.05 0.5 0.05"/>
+            </geometry>
+            <material name="orange"/>
+        </visual>
+        <collision>
+            <origin xyz="0 0 ${wheel_offset_z}"/>
+            <geometry>
+                <box size="0.05 0.5 0.05"/>
+            </geometry>
+        </collision>
+        <xacro:inertial_box mass="0.5" x="0.05" y="0.5" z="0.05">
+            <origin xyz="0 0 ${wheel_offset_z}" rpy="0 0 0"/>
+        </xacro:inertial_box>
+    </link>
     </xacro:macro>
 </robot>

Commit message: changed type of back wheels to "continous" in urdf

File: description/ros2_control/diffbot.ros2_control.xacro (robot description, xacro)
@@ -47,4 +47,14 @@
           <state_interface name="velocity"/>
         </joint>
+        <joint name="${prefix}back_left_wheel_joint">
+          <command_interface name="velocity"/>
+          <state_interface name="position"/>
+          <state_interface name="velocity"/>
+        </joint>
+        <joint name="${prefix}back_right_wheel_joint">
+          <command_interface name="velocity"/>
+          <state_interface name="position"/>
+          <state_interface name="velocity"/>
+        </joint>
       </ros2_control>
       <gazebo reference="imu_link">

File: description/urdf/diffbot_description.urdf.xacro (robot description, xacro)
@@ -341,5 +341,5 @@
         <parent link="base_link"/>
         <child link="left_wheel"/>
-        <origin xyz="${front_wheel_offset_x} -${wheel_offset_y} 0" rpy="-${pi/2} 0 0" />
+        <origin xyz="${front_wheel_offset_x} ${wheel_offset_y} 0" rpy="-${pi/2} 0 0" />
         <axis xyz="0 0 1"/>
     </joint>
@@ -355,4 +355,13 @@
                 <sphere radius="${wheel_radius}"/>
             </geometry>
+            <surface>
+                <friction>
+                    <torsional>
+                        <coefficient>=0.5</coefficient>
+                        <use_patch_radius>false</use_patch_radius>
+                        <surface_radius>${wheel_radius}</surface_radius>
+                    </torsional>
+                </friction>
+            </surface>
         </collision>
         <xacro:inertial_cylinder mass="${wheel_mass}" length="${wheel_thickness}" radius="${wheel_radius}">
@@ -367,5 +376,5 @@
         <parent link="base_link"/>
         <child link="right_wheel"/>
-        <origin xyz="${front_wheel_offset_x} ${wheel_offset_y} 0" rpy="${pi/2} 0 0" />
+        <origin xyz="${front_wheel_offset_x} -${wheel_offset_y} 0" rpy="${pi/2} 0 0" />
         <axis xyz="0 0 -1"/>
     </joint>
@@ -381,4 +390,13 @@
                 <sphere radius="${wheel_radius}"/>
             </geometry>
+            <surface>
+                <friction>
+                    <torsional>
+                        <coefficient>0.5</coefficient>
+                        <use_patch_radius>false</use_patch_radius>
+                        <surface_radius>${wheel_radius}</surface_radius>
+                    </torsional>
+                </friction>
+            </surface>
         </collision>
         <xacro:inertial_cylinder mass="${wheel_mass}" length="${wheel_thickness}" radius="${wheel_radius}">
@@ -390,5 +408,5 @@
     </gazebo>
     <!-- BACK LEFT WHEEL LINK -->
-    <joint name="back_left_wheel_joint" type="fixed">
+    <joint name="back_left_wheel_joint" type="continuous">
         <parent link="base_link"/>
         <child link="back_left_wheel"/>
@@ -407,4 +425,9 @@
                 <sphere radius="${wheel_radius}"/>
             </geometry>
+            <torsional>
+                <coefficient>0.5</coefficient>
+                <use_patch_radius>false</use_patch_radius>
+                <surface_radius>${wheel_radius}</surface_radius>
+            </torsional>
         </collision>
         <xacro:inertial_cylinder mass="${caster_wheel_mass}" length="${wheel_thickness}" radius="${wheel_radius}">
@@ -418,5 +441,5 @@
     </gazebo>
     <!-- BACK RIGHT WHEEL LINK -->
-    <joint name="back_right_wheel_joint" type="fixed">
+    <joint name="back_right_wheel_joint" type="continuous">
         <parent link="base_link"/>
         <child link="back_right_wheel"/>
@@ -435,4 +458,9 @@
                 <sphere radius="${wheel_radius}"/>
             </geometry>
+            <torsional>
+                <coefficient>0.5</coefficient>
+                <use_patch_radius>false</use_patch_radius>
+                <surface_radius>${wheel_radius}</surface_radius>
+            </torsional>
         </collision>
         <xacro:inertial_cylinder mass="${caster_wheel_mass}" length="${wheel_thickness}" radius="${wheel_radius}">
