Commit message: update angular velocity and acceleration

File: description/urdf/depth_camera.xacro (robot description, xacro)
@@ -1,21 +1,21 @@
 <?xml version="1.0"?>
 <robot xmlns:xacro="http://www.ros.org/wiki/xacro" >
-    <xacro:property name="chassis_length" value="1.35" />
-    <xacro:property name="chassis_width" value="0.5" />
-    <xacro:property name="chassis_height" value="0.01" />
-    <xacro:property name="chassis_mass" value="1.0" />
+    <xacro:property name="chassis_length" value="1.3501" />
+    <xacro:property name="chassis_to_base_link" value="0.73595" />
+    <xacro:property name="profile_height" value="0.0254" />
+    <xacro:property name="profile_width" value="0.0254" />
+    <xacro:property name="tower_height" value="0.508" />
     <xacro:property name="wheel_radius" value="0.1778" />
     <xacro:property name="wheel_thickness" value="0.07" />
     <xacro:property name="wheel_mass" value="0.05" />
-    <xacro:property name="wheel_offset_x" value="0.2135" />
-    <xacro:property name="wheel_offset_y" value="0.285" />
-    <xacro:property name="wheel_offset_z" value="0.01" />
-    <xacro:property name="caster_wheel_radius" value="0.1778"/>
+    <xacro:property name="front_wheel_offset_x" value="0.3876" />
+    <xacro:property name="back_wheel_offset_x" value="0.437" />
+    <xacro:property name="wheel_offset_y" value="0.3182" />
+    <xacro:property name="wheel_offset_z" value="0.1778" />
     <xacro:property name="caster_wheel_mass" value="0.01"/>
-    <xacro:property name="caster_wheel_offset_x" value="1.1365" />
     <joint name="camera_joint" type="fixed">
         <parent link="base_link"/>
         <child link="camera_link"/>
-        <origin xyz="${caster_wheel_offset_x-0.1} 0 0.075" rpy="0 0 0"/>
+        <origin xyz="0.3879 0 0.075" rpy="0 0 0"/>
     </joint>
     <link name="camera_link">

File: description/urdf/lidar.xacro (robot description, xacro)
@@ -1,21 +1,21 @@
 <?xml version="1.0"?>
 <robot xmlns:xacro="http://www.ros.org/wiki/xacro" >
-    <xacro:property name="chassis_length" value="1.35" />
-    <xacro:property name="chassis_width" value="0.5" />
-    <xacro:property name="chassis_height" value="0.01" />
-    <xacro:property name="chassis_mass" value="1.0" />
+    <xacro:property name="chassis_length" value="1.3501" />
+    <xacro:property name="chassis_to_base_link" value="0.73595" />
+    <xacro:property name="profile_height" value="0.0254" />
+    <xacro:property name="profile_width" value="0.0254" />
+    <xacro:property name="tower_height" value="0.508" />
     <xacro:property name="wheel_radius" value="0.1778" />
     <xacro:property name="wheel_thickness" value="0.07" />
     <xacro:property name="wheel_mass" value="0.05" />
-    <xacro:property name="wheel_offset_x" value="0.2135" />
-    <xacro:property name="wheel_offset_y" value="0.285" />
-    <xacro:property name="wheel_offset_z" value="0.01" />
-    <xacro:property name="caster_wheel_radius" value="0.1778"/>
+    <xacro:property name="front_wheel_offset_x" value="0.3876" />
+    <xacro:property name="back_wheel_offset_x" value="0.437" />
+    <xacro:property name="wheel_offset_y" value="0.3182" />
+    <xacro:property name="wheel_offset_z" value="0.1778" />
     <xacro:property name="caster_wheel_mass" value="0.01"/>
-    <xacro:property name="caster_wheel_offset_x" value="1.1365" />
     <joint name="laser_joint" type="fixed">
-        <parent link="base_footprint"/>
+        <parent link="base_link"/>
         <child link="laser_frame"/>
-        <origin xyz="0.465 0 ${0.435+0.05}" rpy="0 0 0"/>
+        <origin xyz="0 0 ${tower_height-profile_width +profile_height*2 }" rpy="0 0 0"/>
     </joint>
     <link name="laser_frame">
@@ -56,5 +56,5 @@
             <plugin name="laser_controller" filename="libgazebo_ros_ray_sensor.so">
                 <ros>
-                    <argument>~/out:=scan</argument>
+                    <argument>~/out:=laser</argument>
                 </ros>
                 <output_type>sensor_msgs/LaserScan</output_type>

File: description/urdf/robot_core.xacro (robot description, xacro)
@@ -1,9 +1,5 @@
 <?xml version="1.0"?>
 <robot xmlns:xacro="http://www.ros.org/wiki/xacro" >
-    <!-- the copy of robot_core_1 urdf -->
-    <xacro:macro name="diffbot" params="prefix">
     <xacro:include filename="inertial_macros.xacro"/>
-    <xacro:include filename="lidar.xacro" />
-    <xacro:include filename="depth_camera.xacro"/>
     <xacro:property name="chassis_length" value="1.3501" />
     <xacro:property name="chassis_to_base_link" value="0.73595" />
@@ -19,4 +15,19 @@
     <xacro:property name="wheel_offset_z" value="0.1778" />
     <xacro:property name="caster_wheel_mass" value="0.01"/>
+    <material name="white">
+        <color rgba="1 1 1 1" />
+    </material>
+    <material name="orange">
+        <color rgba="1 0.3 0.1 1"/>
+    </material>
+    <material name="blue">
+        <color rgba="0.2 0.2 1 1"/>
+    </material>
+    <material name="black">
+        <color rgba="0 0 0 1"/>
+    </material>
+    <material name="red">
+        <color rgba="1 0 0 1"/>
+    </material>
     <!-- BASE LINK -->
     <link name="base_link">
@@ -30,10 +41,4 @@
     <link name="base_footprint">
     </link>
-    <joint name="imu_joint" type="fixed">
-        <parent link="base_link" />
-        <child link="imu_link" />
-        <origin xyz="0 0 0" rpy="0 0 0" />
-    </joint>
-    <link name="imu_link" />
     <!-- CHASSIS LONG BASE LEFT -->
     <!-- Needs to be 1.35m long, to the left by 0.2604m -->
@@ -445,4 +450,3 @@
         <mu2 value="0.001"/>
     </gazebo>
-    </xacro:macro>
 </robot>

Commit message: update the new config of robot

File: description/urdf/depth_camera.xacro (robot description, xacro)
@@ -2,20 +2,27 @@
 <robot xmlns:xacro="http://www.ros.org/wiki/xacro" >
     <xacro:property name="chassis_length" value="1.3501" />
-    <xacro:property name="chassis_to_base_link" value="0.73595" />
+    <xacro:property name="chassis_to_base_link" value="0.4954" />
     <xacro:property name="profile_height" value="0.0254" />
     <xacro:property name="profile_width" value="0.0254" />
-    <xacro:property name="tower_height" value="0.508" />
+    <xacro:property name="tower_height" value="0.388" />
     <xacro:property name="wheel_radius" value="0.1778" />
     <xacro:property name="wheel_thickness" value="0.07" />
-    <xacro:property name="wheel_mass" value="0.05" />
-    <xacro:property name="front_wheel_offset_x" value="0.3876" />
-    <xacro:property name="back_wheel_offset_x" value="0.437" />
+    <xacro:property name="wheel_mass" value="56" />
+    <xacro:property name="front_wheel_offset_x" value="0.14" />
+    <xacro:property name="back_wheel_offset_x" value="0.49" />
     <xacro:property name="wheel_offset_y" value="0.3182" />
     <xacro:property name="wheel_offset_z" value="0.1778" />
-    <xacro:property name="caster_wheel_mass" value="0.01"/>
+    <xacro:property name="caster_wheel_mass" value="56"/>
+    <xacro:property name="double_prof_mass" value="0.235398773"/>
+    <xacro:property name="single_prof_mass" value="0.147601476"/>
+    <xacro:property name="spoke_mass" value="1.6"/>
+    <xacro:property name="motorgearbox_mass" value="136"/>
+    <xacro:property name="scoop_mass" value="196"/>
+    <xacro:property name="tiltingact_mass" value="38"/>
+    <xacro:property name="liftingact_mass" value="44"/>
     <joint name="camera_joint" type="fixed">
         <parent link="base_link"/>
         <child link="camera_link"/>
-        <origin xyz="0.3879 0 0.075" rpy="0 0 0"/>
+        <origin xyz="0 0 ${tower_height-profile_width +profile_height*2}" rpy="0 0 0"/>
     </joint>
     <link name="camera_link">

File: description/urdf/diffbot.urdf.xacro (robot description, xacro)
@@ -5,6 +5,6 @@
   <xacro:arg name="sim_mode" default="false"/>
   <!-- <xacro:include filename="$(find diffdrive_arduino)/urdf/diffbot_description.urdf.xacro" /> -->
-  <xacro:include filename="$(find ros_phoenix)/urdf/diffbot_description.urdf.xacro" />
-  <!-- <xacro:include filename="$(find ros_phoenix)/urdf/robot_core.urdf.xacro" /> -->
+  <!-- <xacro:include filename="$(find ros_phoenix)/urdf/diffbot_description.urdf.xacro" /> -->
+  <xacro:include filename="$(find ros_phoenix)/urdf/robot_core.urdf.xacro" />
   <!-- Import Rviz colors -->
   <!-- <xacro:include filename="$(find diffdrive_arduino)/urdf/diffbot.materials.xacro" /> -->

File: description/urdf/diffbot_description.urdf.xacro (robot description, xacro)
@@ -358,5 +358,5 @@
                 <friction>
                     <torsional>
-                        <coefficient>=0.5</coefficient>
+                        <coefficient>1.0</coefficient>
                         <use_patch_radius>false</use_patch_radius>
                         <surface_radius>${wheel_radius}</surface_radius>
@@ -393,5 +393,5 @@
                 <friction>
                     <torsional>
-                        <coefficient>0.5</coefficient>
+                        <coefficient>1.0</coefficient>
                         <use_patch_radius>false</use_patch_radius>
                         <surface_radius>${wheel_radius}</surface_radius>
@@ -425,9 +425,11 @@
                 <sphere radius="${wheel_radius}"/>
             </geometry>
-            <torsional>
-                <coefficient>0.5</coefficient>
-                <use_patch_radius>false</use_patch_radius>
-                <surface_radius>${wheel_radius}</surface_radius>
-            </torsional>
+            <friction>
+                <torsional>
+                    <coefficient>1.0</coefficient>
+                    <use_patch_radius>false</use_patch_radius>
+                    <surface_radius>${wheel_radius}</surface_radius>
+                </torsional>
+            </friction>
         </collision>
         <xacro:inertial_cylinder mass="${caster_wheel_mass}" length="${wheel_thickness}" radius="${wheel_radius}">
@@ -458,9 +460,11 @@
                 <sphere radius="${wheel_radius}"/>
             </geometry>
-            <torsional>
-                <coefficient>0.5</coefficient>
-                <use_patch_radius>false</use_patch_radius>
-                <surface_radius>${wheel_radius}</surface_radius>
-            </torsional>
+            <friction>
+                <torsional>
+                    <coefficient>1.0</coefficient>
+                    <use_patch_radius>false</use_patch_radius>
+                    <surface_radius>${wheel_radius}</surface_radius>
+                </torsional>
+            </friction>
         </collision>
         <xacro:inertial_cylinder mass="${caster_wheel_mass}" length="${wheel_thickness}" radius="${wheel_radius}">

File: description/urdf/lidar.xacro (robot description, xacro)
@@ -2,20 +2,27 @@
 <robot xmlns:xacro="http://www.ros.org/wiki/xacro" >
     <xacro:property name="chassis_length" value="1.3501" />
-    <xacro:property name="chassis_to_base_link" value="0.73595" />
+    <xacro:property name="chassis_to_base_link" value="0.4954" />
     <xacro:property name="profile_height" value="0.0254" />
     <xacro:property name="profile_width" value="0.0254" />
-    <xacro:property name="tower_height" value="0.508" />
+    <xacro:property name="tower_height" value="0.388" />
     <xacro:property name="wheel_radius" value="0.1778" />
     <xacro:property name="wheel_thickness" value="0.07" />
-    <xacro:property name="wheel_mass" value="0.05" />
-    <xacro:property name="front_wheel_offset_x" value="0.3876" />
-    <xacro:property name="back_wheel_offset_x" value="0.437" />
+    <xacro:property name="wheel_mass" value="56" />
+    <xacro:property name="front_wheel_offset_x" value="0.14" />
+    <xacro:property name="back_wheel_offset_x" value="0.49" />
     <xacro:property name="wheel_offset_y" value="0.3182" />
     <xacro:property name="wheel_offset_z" value="0.1778" />
-    <xacro:property name="caster_wheel_mass" value="0.01"/>
+    <xacro:property name="caster_wheel_mass" value="56"/>
+    <xacro:property name="double_prof_mass" value="0.235398773"/>
+    <xacro:property name="single_prof_mass" value="0.147601476"/>
+    <xacro:property name="spoke_mass" value="1.6"/>
+    <xacro:property name="motorgearbox_mass" value="136"/>
+    <xacro:property name="scoop_mass" value="196"/>
+    <xacro:property name="tiltingact_mass" value="38"/>
+    <xacro:property name="liftingact_mass" value="44"/>
     <joint name="laser_joint" type="fixed">
         <parent link="base_link"/>
         <child link="laser_frame"/>
-        <origin xyz="0 0 ${tower_height-profile_width +profile_height*2 }" rpy="0 0 0"/>
+        <origin xyz="0 0 ${tower_height-profile_width +profile_height*2 +0.03 }" rpy="0 0 0"/>
     </joint>
     <link name="laser_frame">
@@ -33,5 +40,5 @@
         <xacro:inertial_cylinder mass="0.1" length="0.04" radius="0.05">
             <origin xyz="0 0 0" rpy="0 0 0"/>
-        </xacro:inertial_cylinder>
+        </xacro:inertial_cylinder>1
     </link>
     <gazebo reference="laser_frame">
