Commit message: update the new config of robot

File: description/urdf/robot_core.urdf.xacro (robot description, xacro)
@@ -1,72 +1,471 @@
 <?xml version="1.0"?>
 <robot xmlns:xacro="http://www.ros.org/wiki/xacro" >
+    <!-- the copy of robot_core_1 urdf -->
     <xacro:macro name="diffbot" params="prefix">
     <xacro:include filename="inertial_macros.xacro"/>
-    <xacro:include filename="lidar.xacro" />
+    <!-- <xacro:include filename="lidar-3d.urdf.xacro" /> -->
     <xacro:include filename="depth_camera.xacro"/>
-    <!-- inlucde bracket -->
-    <!-- <xacro:include filename="$(find ros_phoenix)/urdf/brackets.xacro" /> -->
-    <xacro:property name="chassis_length" value="1.35" />
-    <xacro:property name="chassis_width" value="0.5" />
-    <xacro:property name="chassis_height" value="0.01" />
-    <xacro:property name="chassis_mass" value="1.0" />
+    <xacro:include filename="lidar.xacro"/>
+    <xacro:property name="chassis_length" value="1.3501" />
+    <xacro:property name="chassis_to_base_link" value="0.4954" />
+    <xacro:property name="profile_height" value="0.0254" />
+    <xacro:property name="profile_width" value="0.0254" />
+    <xacro:property name="tower_height" value="0.388" />
     <xacro:property name="wheel_radius" value="0.1778" />
     <xacro:property name="wheel_thickness" value="0.07" />
-    <xacro:property name="wheel_mass" value="0.05" />
-    <xacro:property name="wheel_offset_x" value="0.2135" />
-    <xacro:property name="wheel_offset_y" value="0.285" />
-    <xacro:property name="wheel_offset_z" value="0.01" />
-    <xacro:property name="caster_wheel_radius" value="0.1778"/>
-    <xacro:property name="caster_wheel_mass" value="0.01"/>
-    <xacro:property name="caster_wheel_offset_x" value="1.1365" />
+    <xacro:property name="wheel_mass" value="56" />
+    <xacro:property name="front_wheel_offset_x" value="0.14" />
+    <xacro:property name="back_wheel_offset_x" value="0.49" />
+    <xacro:property name="wheel_offset_y" value="0.3182" />
+    <xacro:property name="wheel_offset_z" value="0.1778" />
+    <xacro:property name="caster_wheel_mass" value="56"/>
+    <xacro:property name="double_prof_mass" value="0.235398773"/>
+    <xacro:property name="single_prof_mass" value="0.147601476"/>
+    <xacro:property name="spoke_mass" value="1.6"/>
+    <xacro:property name="motorgearbox_mass" value="136"/>
+    <xacro:property name="scoop_mass" value="196"/>
+    <xacro:property name="tiltingact_mass" value="38"/>
+    <xacro:property name="liftingact_mass" value="44"/>
     <!-- BASE LINK -->
     <link name="base_link">
     </link>
-    <joint name="imu_joint" type="fixed">
-        <parent link="base_footprint" />
-        <child link="imu_link" />
-        <origin xyz="0 0.05 ${wheel_offset_x+0.042}" rpy="0 0 0" />
-    </joint>
-    <link name="imu_link" />
     <!-- BASE_FOOTPRINT LINK -->
     <joint name="base_footprint_joint" type="fixed">
     	<parent link="base_link"/>
     	<child link="base_footprint"/>
-    	<origin xyz="0 0 0" rpy="${pi} ${pi} 0"/>
+    	<origin xyz="0 0 0" rpy="0 0 0"/>
     </joint>
     <link name="base_footprint">
     </link>
-    <!-- CHASSIS LINK -->
-    <joint name="chassis_joint" type="fixed">
-        <parent link="base_footprint"/>
-        <child link="chassis"/>
-        <origin xyz="${-wheel_offset_x} 0 ${-wheel_offset_z}"/>
-    </joint>
-    <link name="chassis">
-        <visual>
-            <origin xyz="${chassis_length/2} 0 ${chassis_height/2}"/>
-            <geometry>
-                <box size="${chassis_length} ${chassis_width} ${chassis_height}"/>
-            </geometry>
-            <material name="white"/>
-        </visual>
-        <collision>
-            <origin xyz="${chassis_length/2} 0 ${chassis_height/2}"/>
-            <geometry>
-                <box size="${chassis_length} ${chassis_width} ${chassis_height}"/>
-            </geometry>
-        </collision>
-        <xacro:inertial_box mass="0.5" x="${chassis_length}" y="${chassis_width}" z="${chassis_height}">
-            <origin xyz="${chassis_length/2} 0 ${chassis_height/2}" rpy="0 0 0"/>
-        </xacro:inertial_box>
-    </link>
-    <gazebo reference="chassis">
-        <material>Gazebo/White</material>
-    </gazebo>
-    <!-- BACK LEFT WHEEL LINK -->
+    <joint name="imu_joint" type="fixed">
+        <parent link="base_link" />
+        <child link="imu_link" />
+        <origin xyz="0 0 ${tower_height-profile_width +profile_height*2 + 0.06}" rpy="0 0 0" />
+    </joint>
+    <link name="imu_link">
+        <visual>
+            <geometry>
+                <box size="0.03 0.02 0.01"/>
+            </geometry>
+            <material name="orange"/>
+        </visual>
+    </link>
+    <!-- CHASSIS LONG BASE LEFT -->
+    <!-- Needs to be 1.35m long, to the left by 0.2604m -->
+    <joint name="chassis_base_left" type="fixed">
+        <parent link="base_link"/>
+        <child link="chassis_base_left"/>
+        <origin xyz="${chassis_to_base_link} -0.2604 0"/>
+    </joint>
+    <link name="chassis_base_left">
+        <visual>
+            <origin xyz="${-chassis_length/2} 0 0"/>
+            <geometry>
+                <box size="${chassis_length} 0.0508 ${profile_height}"/>
+            </geometry>
+            <material name="white"/>
+        </visual>
+        <collision>
+            <origin xyz="${-chassis_length/2} 0 0"/>
+            <geometry>
+                <box size="${chassis_length} 0.0508 ${profile_height}"/>
+            </geometry>
+        </collision>
+        <xacro:inertial_box mass="${double_prof_mass*chassis_length*100}" x="${-chassis_length}" y="0.0508" z="${profile_height}">
+            <origin xyz="${chassis_length/2} 0 0" rpy="0 0 0"/>
+        </xacro:inertial_box>
+    </link>
+    <gazebo reference="chassis_base_left">
+        <material>Gazebo/White</material>
+    </gazebo>
+    <!-- CHASSIS LONG BASE RIGHT -->
+    <!-- Needs to be 1.35m long, to the left by  -->
+    <joint name="chassis_base_right" type="fixed">
+        <parent link="base_link"/>
+        <child link="chassis_base_right"/>
+        <origin xyz="${chassis_to_base_link} 0.2604 0"/>
+    </joint>
+    <link name="chassis_base_right">
+        <visual>
+            <origin xyz="${-chassis_length/2} 0 0"/>
+            <geometry>
+                <box size="${chassis_length} 0.0508 ${profile_height}"/>
+            </geometry>
+            <material name="white"/>
+        </visual>
+        <collision>
+            <origin xyz="${-chassis_length/2} 0 0"/>
+            <geometry>
+                <box size="${chassis_length} 0.0508 ${profile_height}"/>
+            </geometry>
+        </collision>
+        <xacro:inertial_box mass="${double_prof_mass*chassis_length*100}" x="${-chassis_length}" y="0.0508" z="${profile_height}">
+            <origin xyz="${chassis_length/2} 0 0" rpy="0 0 0"/>
+        </xacro:inertial_box>
+    </link>
+    <gazebo reference="chassis_base_right">
+        <material>Gazebo/White</material>
+    </gazebo>
+    <!-- TOWER BASE -->
+    <joint name="tower_base_" type="fixed">
+        <parent link="base_link"/>
+        <child link="tower_base"/>
+        <origin xyz="0 0 0"/>
+    </joint>
+    <link name="tower_base">
+        <visual>
+            <origin xyz="0 0 0"/>
+            <geometry>
+                <box size="${profile_width} 0.4702 ${profile_height}"/>
+            </geometry>
+            <material name="white"/>
+        </visual>
+        <collision>
+            <origin xyz="0 0 0"/>
+            <geometry>
+                <box size="${profile_width} 0.4702 ${profile_height}"/>
+            </geometry>
+        </collision>
+        <xacro:inertial_box mass="${single_prof_mass*47.02}" x="${profile_width}" y="0.4702" z="${profile_height}">
+            <origin xyz="0 0 0" rpy="0 0 0"/>
+        </xacro:inertial_box>
+    </link>
+    <gazebo reference="tower_base">
+        <material>Gazebo/White</material>
+    </gazebo>
+    <!-- TOWER MIDDLE -->
+    <joint name="tower_middle_" type="fixed">
+        <parent link="base_link"/>
+        <child link="tower_middle"/>
+        <origin xyz="0 0 0.08"/>
+    </joint>
+    <link name="tower_middle">
+        <visual>
+            <origin xyz="0 0 0"/>
+            <geometry>
+                <box size="${profile_width} 0.4702 ${profile_height}"/>
+            </geometry>
+            <material name="white"/>
+        </visual>
+        <collision>
+            <origin xyz="0 0 0"/>
+            <geometry>
+                <box size="${profile_width} 0.4702 ${profile_height}"/>
+            </geometry>
+        </collision>
+        <xacro:inertial_box mass="${single_prof_mass*47.02}" x="${profile_width}" y="0.4702" z="${profile_height}">
+            <origin xyz="0 0 0" rpy="0 0 0"/>
+        </xacro:inertial_box>
+    </link>
+    <gazebo reference="tower_middle">
+        <material>Gazebo/White</material>
+    </gazebo>
+    <!-- TOWER HEIGHT LEFT -->
+    <!-- Needs to be 0.510m tall -->
+    <joint name="tower_up_left" type="fixed">
+        <parent link="base_link"/>
+        <child link="tower_up_left"/>
+        <origin xyz="0 -0.2478 0"/>
+    </joint>
+    <link name="tower_up_left">
+        <visual>
+            <origin xyz="0 0 ${tower_height/2}"/>
+            <geometry>
+                <box size="${profile_width} ${profile_width} ${tower_height}"/>
+            </geometry>
+            <material name="white"/>
+        </visual>
+        <collision>
+            <origin xyz="0 0 ${tower_height/2}"/>
+            <geometry>
+                <box size="${profile_width} ${profile_width} ${tower_height}"/>
+            </geometry>
+        </collision>
+        <xacro:inertial_box mass="${single_prof_mass*tower_height*100}" x="${profile_width}" y="${profile_width}" z="${tower_height}">
+            <origin xyz="0 0 ${tower_height/2}" rpy="0 0 0"/>
+        </xacro:inertial_box>
+    </link>
+    <gazebo reference="tower_up_left">
+        <material>Gazebo/White</material>
+    </gazebo>
+    <!-- TOWER HEIGHT RIGHT-->
+    <!-- Needs to be 0.510m tall -->
+    <joint name="tower_up_right" type="fixed">
+        <parent link="base_link"/>
+        <child link="tower_up_right"/>
+        <origin xyz="0 0.2478 0"/>
+    </joint>
+    <link name="tower_up_right">
+        <visual>
+            <origin xyz="0 0 ${tower_height/2}"/>
+            <geometry>
+                <box size="${profile_width} ${profile_width} ${tower_height}"/>
+            </geometry>
+            <material name="white"/>
+        </visual>
+        <collision>
+            <origin xyz="0 0 ${tower_height/2}"/>
+            <geometry>
+                <box size="${profile_width} ${profile_width} ${tower_height}"/>
+            </geometry>
+        </collision>
+        <xacro:inertial_box mass="${single_prof_mass*tower_height*100}" x="${profile_width}" y="${profile_width}" z="${tower_height}">
+            <origin xyz="0 0 ${tower_height/2}" rpy="0 0 0"/>
+        </xacro:inertial_box>
+    </link>
+    <gazebo reference="tower_up_right">
+        <material>Gazebo/White</material>
+    </gazebo>
+    <!-- TOWER TOP -->
+    <!-- Needs to be 0.510m tall -->
+    <joint name="tower_top" type="fixed">
+        <parent link="base_link"/>
+        <child link="tower_top"/>
+        <origin xyz="0 0 ${tower_height-profile_width}"/>
+    </joint>
+    <link name="tower_top">
+        <visual>
+            <origin xyz="0 0 0"/>
+            <geometry>
+                <box size="${profile_width} 0.4702 ${profile_height*2}"/>
+            </geometry>
+            <material name="white"/>
+        </visual>
+        <collision>
+            <origin xyz="0 0 0"/>
+            <geometry>
+                <box size="${profile_width} 0.4702 ${profile_height*2}"/>
+            </geometry>
+        </collision>
+        <xacro:inertial_box mass="${double_prof_mass*0.4702*100}" x="${profile_width}" y="0.4702" z="${profile_height*2}">
+            <origin xyz="0 0 0" rpy="0 0 0"/>
+        </xacro:inertial_box>
+    </link>
+    <!-- TOWER SUPPORT LEFT -->
+    <joint name="tower_support_left" type="fixed">
+        <parent link="base_link"/>
+        <child link="tower_support_left"/>
+        <origin xyz="-0.15635 -0.2478 0.160" rpy="0 ${-pi/4} 0"/>
+        <axis xyz="1 0 0"/>
+    </joint>
+    <link name="tower_support_left">
+        <visual>
+            <origin xyz="0 0 0"/>
+            <geometry>
+                <box size="0.4572 ${profile_width} ${profile_height}"/>
+            </geometry>
+            <material name="white"/>
+        </visual>
+        <collision>
+            <origin xyz="0 0 0"/>
+            <geometry>
+                <box size="0.4572 ${profile_width} ${profile_height}"/>
+            </geometry>
+        </collision>
+        <xacro:inertial_box mass="${single_prof_mass*0.4572*100}" x="0.4572" y="${profile_width}" z="${profile_height}">
+            <origin xyz="0 0 0" rpy="0 0 0"/>
+        </xacro:inertial_box>
+    </link>
+    <gazebo reference="tower_support_left">
+        <material>Gazebo/White</material>
+    </gazebo>
+    <!-- TOWER SUPPORT RIGHT -->
+    <joint name="tower_support_right" type="fixed">
+        <parent link="base_link"/>
+        <child link="tower_support_right"/>
+        <origin xyz="-0.15635 0.2478 0.160" rpy="0 ${-pi/4} 0"/>
+        <axis xyz="1 0 0"/>
+    </joint>
+    <link name="tower_support_right">
+        <visual>
+            <origin xyz="0 0 0"/>
+            <geometry>
+                <box size="0.4572 ${profile_width} ${profile_height}"/>
+            </geometry>
+            <material name="white"/>
+        </visual>
+        <collision>
+            <origin xyz="0 0 0"/>
+            <geometry>
+                <box size="0.4572 ${profile_width} ${profile_height}"/>
+            </geometry>
+        </collision>
+        <xacro:inertial_box mass="${single_prof_mass*0.4572*100}" x="0.4572" y="${profile_width}" z="${profile_height}">
+            <origin xyz="0 0 0" rpy="0 0 0"/>
+        </xacro:inertial_box>
+    </link>
+    <gazebo reference="tower_support_right">
+        <material>Gazebo/White</material>
+    </gazebo>
+    <!-- MOTOR BASE FRONT -->
+    <joint name="motor_base_front" type="fixed">
+        <parent link="base_link"/>
+        <child link="motor_base_front"/>
+        <origin xyz="0.1 0 0"/>
+    </joint>
+    <link name="motor_base_front">
+        <visual>
+            <origin xyz="0 0 0"/>
+            <geometry>
+                <box size="${profile_width} 0.4702 ${profile_height}"/>
+            </geometry>
+            <material name="white"/>
+        </visual>
+        <collision>
+            <origin xyz="0 0 0"/>
+            <geometry>
+                <box size="${profile_width} 0.4702 ${profile_height}"/>
+            </geometry>
+        </collision>
+        <xacro:inertial_box mass="${single_prof_mass*0.4702*100}" x="${profile_width}" y="0.4702" z="${profile_height}">
+            <origin xyz="0 0 0" rpy="0 0 0"/>
+        </xacro:inertial_box>
+    </link>
+    <gazebo reference="motor_base_front">
+        <material>Gazebo/White</material>
+    </gazebo>
+    <!-- MOTOR BASE BACK -->
+    <joint name="motor_base_back" type="fixed">
+        <parent link="base_link"/>
+        <child link="motor_base_back"/>
+        <origin xyz="0.175 0 0"/>
+    </joint>
+    <link name="motor_base_back">
+        <visual>
+            <origin xyz="0 0 0"/>
+            <geometry>
+                <box size="${profile_width} 0.4702 ${profile_height}"/>
+            </geometry>
+            <material name="white"/>
+        </visual>
+        <collision>
+            <origin xyz="0 0 0"/>
+            <geometry>
+                <box size="${profile_width} 0.4702 ${profile_height}"/>
+            </geometry>
+        </collision>
+        <xacro:inertial_box mass="${single_prof_mass*0.4702*100}" x="${profile_width}" y="0.4702" z="${profile_height}">
+            <origin xyz="0 0 0" rpy="0 0 0"/>
+        </xacro:inertial_box>
+    </link>
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