Commit message: update

File: description/urdf/depth_camera.xacro (robot description, xacro)
@@ -24,5 +24,5 @@
         <parent link="base_link"/>
         <child link="camera_link"/>
-        <origin xyz="0 0 ${tower_height-profile_width +profile_height*2}" rpy="0 0 0"/>
+        <origin xyz="0.1919 0 0.2016" rpy="0 0 0"/>
     </joint>
     <link name="camera_link">
@@ -42,5 +42,5 @@
     <gazebo reference="camera_link">
         <material>Gazebo/Red</material>
-        <sensor name="camera" type="depth">
+        <sensor name="depth_camera" type="depth">
             <pose> 0 0 0 0 0 0 </pose>
             <visualize>true</visualize>

File: description/urdf/lidar.xacro (robot description, xacro)
@@ -24,5 +24,5 @@
         <parent link="base_link"/>
         <child link="laser_frame"/>
-        <origin xyz="0 0 ${tower_height-profile_width +profile_height*2 +0.03 }" rpy="0 0 0"/>
+        <origin xyz="0.10045 0 ${tower_height-profile_width +profile_height*2 }" rpy="0 0 0"/>
     </joint>
     <link name="laser_frame">
@@ -46,5 +46,5 @@
         <sensor name="laser" type="ray">
             <pose> 0 0 0 0 0 0 </pose>
-            <visualize>true</visualize>
+            <visualize>false</visualize>
             <update_rate>10</update_rate>
             <ray>

File: description/urdf/robot_core.urdf.xacro (robot description, xacro)
@@ -4,7 +4,7 @@
     <xacro:macro name="diffbot" params="prefix">
     <xacro:include filename="inertial_macros.xacro"/>
-    <!-- <xacro:include filename="lidar-3d.urdf.xacro" /> -->
     <xacro:include filename="depth_camera.xacro"/>
     <xacro:include filename="lidar.xacro"/>
+    <!-- <xacro:include filename="lidar_3d.xacro"/> -->
     <xacro:property name="chassis_length" value="1.3501" />
     <xacro:property name="chassis_to_base_link" value="0.4954" />
@@ -41,5 +41,5 @@
         <parent link="base_link" />
         <child link="imu_link" />
-        <origin xyz="0 0 ${tower_height-profile_width +profile_height*2 + 0.06}" rpy="0 0 0" />
+        <origin xyz="0.10045 0 ${tower_height-profile_width +profile_height*2 - 0.02}" rpy="0 0 0" />
     </joint>
     <link name="imu_link">
@@ -603,5 +603,5 @@
         <parent link="base_link"/>
         <child link="doser_left"/>
-        <origin xyz="-0.597 -0.1587525 0.2" rpy="0 ${pi/5.81} 0"/>
+        <origin xyz="-0.647 -0.1587525 0.11" rpy="0 ${pi/5.81} 0"/>
         <axis xyz="1 0 0"/>
     </joint>
@@ -610,15 +610,15 @@
             <origin xyz="0 0 0"/>
             <geometry>
-                <box size="0.4153 0.005 0.307"/>
-            </geometry>
-            <material name="white"/>
-        </visual>
-        <collision>
-            <origin xyz="0 0 0"/>
-            <geometry>
-                <box size="0.4153 0.005 0.307"/>
-            </geometry>
-        </collision>
-        <xacro:inertial_box mass="49" x="0.4153" y="0.005" z="0.307">
+                <box size="0.4153 0.005 0.1"/>
+            </geometry>
+            <material name="white"/>
+        </visual>
+        <collision>
+            <origin xyz="0 0 0"/>
+            <geometry>
+                <box size="0.4153 0.005 0.1"/>
+            </geometry>
+        </collision>
+        <xacro:inertial_box mass="49" x="0.4153" y="0.005" z="0.1">
             <origin xyz="0 0 0" rpy="0 0 0"/>
         </xacro:inertial_box>
@@ -630,5 +630,5 @@
         <parent link="base_link"/>
         <child link="doser_right"/>
-        <origin xyz="-0.597 0.1587525 0.2" rpy="0 ${pi/5.81} 0"/>
+        <origin xyz="-0.647 0.1587525 0.11" rpy="0 ${pi/5.81} 0"/>
         <axis xyz="1 0 0"/>
     </joint>
@@ -637,15 +637,15 @@
             <origin xyz="0 0 0"/>
             <geometry>
-                <box size="0.4153 0.005 0.307"/>
-            </geometry>
-            <material name="white"/>
-        </visual>
-        <collision>
-            <origin xyz="0 0 0"/>
-            <geometry>
-                <box size="0.4153 0.005 0.307"/>
-            </geometry>
-        </collision>
-        <xacro:inertial_box mass="49" x="0.4153" y="0.005" z="0.307">
+                <box size="0.4153 0.005 0.1"/>
+            </geometry>
+            <material name="white"/>
+        </visual>
+        <collision>
+            <origin xyz="0 0 0"/>
+            <geometry>
+                <box size="0.4153 0.005 0.1"/>
+            </geometry>
+        </collision>
+        <xacro:inertial_box mass="49" x="0.4153" y="0.005" z="0.1">
             <origin xyz="0 0 0" rpy="0 0 0"/>
         </xacro:inertial_box>
@@ -769,4 +769,138 @@
         <material>Gazebo/Orange</material>
     </gazebo>
+    <!-- ELECTRICAL BOX -->
+    <joint name="elec_box_base" type="fixed">
+        <parent link="base_link"/>
+        <child link="elec_base"/>
+        <origin xyz="0.10045 0 0.1"/>
+    </joint>
+    <link name="elec_base">
+        <visual>
+            <origin xyz="0 0 0"/>
+            <geometry>
+                <box size="0.1829 0.3988 0.019"/>
+            </geometry>
+            <material name="orange"/>
+        </visual>
+        <collision>
+            <origin xyz="0 0 0"/>
+            <geometry>
+                <box size="0.1829 0.3988 0.019"/>
+            </geometry>
+        </collision>
+        <xacro:inertial_box mass="20" x="0.1829" y="0.3988" z="0.019">
+            <origin xyz="0 0 0" rpy="0 0 0"/>
+        </xacro:inertial_box>
+    </link>
+    <gazebo reference="elec_base">
+        <material>Gazebo/White</material>
+    </gazebo>
+    <joint name="elec_box_top" type="fixed">
+        <parent link="base_link"/>
+        <child link="elec_top"/>
+        <origin xyz="0.10045 0 0.3616"/>
+    </joint>
+    <link name="elec_top">
+        <visual>
+            <origin xyz="0 0 0"/>
+            <geometry>
+                <box size="0.1829 0.3988 0.019"/>
+            </geometry>
+            <material name="orange"/>
+        </visual>
+        <collision>
+            <origin xyz="0 0 0"/>
+            <geometry>
+                <box size="0.1829 0.3988 0.019"/>
+            </geometry>
+        </collision>
+        <xacro:inertial_box mass="20" x="0.1829" y="0.3988" z="0.019">
+            <origin xyz="0 0 0" rpy="0 0 0"/>
+        </xacro:inertial_box>
+    </link>
+    <gazebo reference="elec_top">
+        <material>Gazebo/White</material>
+    </gazebo>
+    <joint name="elec_box_left" type="fixed">
+        <parent link="base_link"/>
+        <child link="elec_left"/>
+        <origin xyz="0.10045 -0.1995 0.23095"/>
+    </joint>
+    <link name="elec_left">
+        <visual>
+            <origin xyz="0 0 0"/>
+            <geometry>
+                <box size="0.1829 0.009 0.28"/>
+            </geometry>
+            <material name="orange"/>
+        </visual>
+        <collision>
+            <origin xyz="0 0 0"/>
+            <geometry>
+                <box size="0.1829 0.009 0.28"/>
+            </geometry>
+        </collision>
+        <xacro:inertial_box mass="20" x="0.1829" y="0.009" z="0.28">
+            <origin xyz="0 0 0" rpy="0 0 0"/>
+        </xacro:inertial_box>
+    </link>
+    <gazebo reference="elec_left">
+        <material>Gazebo/White</material>
+    </gazebo>
+    <joint name="elec_box_right" type="fixed">
+        <parent link="base_link"/>
+        <child link="elec_right"/>
+        <origin xyz="0.10045 0.1995 0.23095"/>
+    </joint>
+    <link name="elec_right">
+        <visual>
+            <origin xyz="0 0 0"/>
+            <geometry>
+                <box size="0.1829 0.009 0.28"/>
+            </geometry>
+            <material name="orange"/>
+        </visual>
+        <collision>
+            <origin xyz="0 0 0"/>
+            <geometry>
+                <box size="0.1829 0.009 0.28"/>
+            </geometry>
+        </collision>
+        <xacro:inertial_box mass="20" x="0.1829" y="0.009" z="0.28">
+            <origin xyz="0 0 0" rpy="0 0 0"/>
+        </xacro:inertial_box>
+    </link>
+    <gazebo reference="elec_right">
+        <material>Gazebo/White</material>
+    </gazebo>
+    <joint name="elec_box_back" type="fixed">
+        <parent link="base_link"/>
+        <child link="elec_back"/>
+        <origin xyz="0.0135 0 0.23095"/>
+    </joint>
+    <link name="elec_back">
+        <visual>
+            <origin xyz="0 0 0"/>
+            <geometry>
+                <box size="0.009 0.3988 0.28"/>
+            </geometry>
+            <material name="orange"/>
+        </visual>
+        <collision>
+            <origin xyz="0 0 0"/>
+            <geometry>
+                <box size="0.009 0.3988 0.28"/>
+            </geometry>
+        </collision>
+        <xacro:inertial_box mass="20" x="0.009" y="0.3988" z="0.28">
+            <origin xyz="0 0 0" rpy="0 0 0"/>
+        </xacro:inertial_box>
+    </link>
+    <gazebo reference="elec_back">
+        <material>Gazebo/White</material>
+    </gazebo>
+    <gazebo reference="actuator_right">
+        <material>Gazebo/Orange</material>
+    </gazebo>
     </xacro:macro>
 </robot>
